File: pi_hat/raspberrypi-gpio-40pin.kicad_pcb (KiCad board)
At the start: 2 copper layers, 65 x 56 mm, 5 parts, among them P1 Conn_02x20_Odd_Even

Commit message: updated schematic, improved layout
Parts:
- added C1: 10uF, Capacitor_SMD:C_0805_2012Metric_Pad1.15x1.40mm_HandSolder, F.Cu at (107.3, 89.0)
- added C10: 0.1uF, Capacitor_SMD:C_0805_2012Metric_Pad1.15x1.40mm_HandSolder, F.Cu at (116.8, 90.8)
- added C11: 0.1uF, Capacitor_SMD:C_0805_2012Metric_Pad1.15x1.40mm_HandSolder, F.Cu at (130.1, 75.1)
- added C12: 0.1uF, Capacitor_SMD:C_0805_2012Metric_Pad1.15x1.40mm_HandSolder, F.Cu at (186.0, 132.2)
- added C13: 0.1uF, Capacitor_SMD:C_0805_2012Metric_Pad1.15x1.40mm_HandSolder, F.Cu at (189.8, 132.2)
- added C14: 0.1uF, Capacitor_SMD:C_0805_2012Metric_Pad1.15x1.40mm_HandSolder, F.Cu at (193.7, 132.2)
- added C15: 0.1uF, Capacitor_SMD:C_0805_2012Metric_Pad1.15x1.40mm_HandSolder, F.Cu at (212.7, 122.1)
- added C16: 0.1uF, Capacitor_SMD:C_0805_2012Metric_Pad1.15x1.40mm_HandSolder, F.Cu at (212.7, 119.5)
- added C17: 0.1uF, Capacitor_SMD:C_0805_2012Metric_Pad1.15x1.40mm_HandSolder, F.Cu at (212.7, 115.7)
- added C18: 100uF, Capacitor_THT:CP_Radial_D6.3mm_P2.50mm, F.Cu at (245.7, 158.9)
- added C19: 100uF, Capacitor_THT:CP_Radial_D6.3mm_P2.50mm, F.Cu at (222.9, 158.9)
- added C2: 10uF, Capacitor_SMD:C_0805_2012Metric_Pad1.15x1.40mm_HandSolder, F.Cu at (119.4, 74.1)
- added C20: 100uF, Capacitor_THT:CP_Radial_D6.3mm_P2.50mm, F.Cu at (196.2, 157.6)
- added C21: 0.1uF, Capacitor_SMD:C_0805_2012Metric_Pad1.15x1.40mm_HandSolder, F.Cu at (197.5, 100.5)
- added C22: 0.1uF, Capacitor_SMD:C_0805_2012Metric_Pad1.15x1.40mm_HandSolder, F.Cu at (193.7, 100.5)
- added C23: 0.1uF, Capacitor_SMD:C_0805_2012Metric_Pad1.15x1.40mm_HandSolder, F.Cu at (189.8, 100.5)
- added C24: 0.1uF, Capacitor_SMD:C_0805_2012Metric_Pad1.15x1.40mm_HandSolder, F.Cu at (178.4, 117.0)
- added C25: 0.1uF, Capacitor_SMD:C_0805_2012Metric_Pad1.15x1.40mm_HandSolder, F.Cu at (178.4, 120.8)
- added C26: 0.1uF, Capacitor_SMD:C_0805_2012Metric_Pad1.15x1.40mm_HandSolder, F.Cu at (178.4, 124.6)
- added C27: 0.1uF, Capacitor_SMD:C_0805_2012Metric_Pad1.15x1.40mm_HandSolder, F.Cu at (161.9, 99.2)
- added C28: 0.1uF, Capacitor_SMD:C_0805_2012Metric_Pad1.15x1.40mm_HandSolder, F.Cu at (161.9, 109.4)
- added C29: 0.1uF, Capacitor_SMD:C_0805_2012Metric_Pad1.15x1.40mm_HandSolder, F.Cu at (163.2, 123.3)
- added C3: 0.1uF, Capacitor_SMD:C_0805_2012Metric_Pad1.15x1.40mm_HandSolder, F.Cu at (107.3, 86.1)
- added C4: 0.1uF, Capacitor_SMD:C_0805_2012Metric_Pad1.15x1.40mm_HandSolder, F.Cu at (130.1, 63.3)
- added C5: 4.7uF, Capacitor_SMD:C_0805_2012Metric_Pad1.15x1.40mm_HandSolder, F.Cu at (149.2, 151.3)
- added C6: 4.7uF, Capacitor_SMD:C_0805_2012Metric_Pad1.15x1.40mm_HandSolder, F.Cu at (149.2, 138.6)
- added C7: 4.7uF, Capacitor_SMD:C_0805_2012Metric_Pad1.15x1.40mm_HandSolder, F.Cu at (164.4, 138.6)
- added C8: 4.7uF, Capacitor_SMD:C_0805_2012Metric_Pad1.15x1.40mm_HandSolder, F.Cu at (164.4, 150.0)
- added C9: 0.1uF, Capacitor_SMD:C_0805_2012Metric_Pad1.15x1.40mm_HandSolder, F.Cu at (112.0, 90.9)
- added D1: 50V_1A, Diode_SMD:D_SMA_Handsoldering, F.Cu at (85.7, 105.5)
- added D2: BLUE, LED_SMD:LED_0805_2012Metric_Pad1.15x1.40mm_HandSolder, F.Cu at (224.1, 113.2)
- added D3: BLUE, LED_SMD:LED_0805_2012Metric_Pad1.15x1.40mm_HandSolder, F.Cu at (224.1, 117.0)
- added D4: BLUE, LED_SMD:LED_0805_2012Metric_Pad1.15x1.40mm_HandSolder, F.Cu at (224.1, 120.8)
- added D5: BLUE, LED_SMD:LED_0805_2012Metric_Pad1.15x1.40mm_HandSolder, F.Cu at (224.1, 124.6)
- added D6: 50V_1A, Diode_SMD:D_SMA_Handsoldering, F.Cu at (235.6, 113.2)
- added D7: 50V_1A, Diode_SMD:D_SMA_Handsoldering, F.Cu at (235.6, 118.2)
- added D8: 50V_1A, Diode_SMD:D_SMA_Handsoldering, F.Cu at (235.6, 123.3)
- added D9: STPS1545D, Package_TO_SOT_THT:TO-220-2_Vertical, F.Cu at (257.1, 141.1)
- added F1: 30A, footprints:MCCQ-121, F.Cu at (247.0, 124.6)
- added F2: 2A, footprints:littlefuse_448, F.Cu at (248.3, 108.1)
- added F3: 4A, footprints:littlefuse_448, F.Cu at (248.3, 103.0)
- added J1: MC000052, footprints:MC000052, F.Cu at (257.1, 127.1)
- added J2: 10pinIDC, Connector_IDC:IDC-Header_2x05_P2.54mm_Vertical, F.Cu at (227.9, 104.3)
- added J3: MOLEX_2031, Connector_Molex:Molex_KK-254_AE-6410-03A_1x03_P2.54mm_Vertical, F.Cu at (236.8, 104.9)
- added JP1: Jumper, Connector_PinHeader_2.54mm:PinHeader_1x02_P2.54mm_Vertical, F.Cu at (73.0, 58.8)
- added JP2: Jumper, Connector_PinHeader_2.54mm:PinHeader_1x02_P2.54mm_Vertical, F.Cu at (153.7, 102.0)
- added MX1: X_STEPPER, footprints:TMC2130, F.Cu at (248.3, 141.1)
- added MX2: MOLEX_2041, Connector_Molex:Molex_KK-254_AE-6410-04A_1x04_P2.54mm_Vertical, F.Cu at (230.5, 160.2)
- added MY1: Y_STEPPER, footprints:TMC2130, F.Cu at (207.6, 153.8)
- added MY2: MOLEX_2041, Connector_Molex:Molex_KK-254_AE-6410-04A_1x04_P2.54mm_Vertical, F.Cu at (207.6, 160.2)
- added MZ1: Z_STEPPER, footprints:TMC2130, F.Cu at (197.5, 141.1)
- added MZ2: MOLEX_2041, Connector_Molex:Molex_KK-254_AE-6410-04A_1x04_P2.54mm_Vertical, F.Cu at (182.2, 158.9)
- added Q1: IRLB8721PBF, Package_TO_SOT_THT:TO-220-3_Vertical, F.Cu at (257.1, 134.8)
- added R1: 100, Resistor_SMD:R_0805_2012Metric_Pad1.15x1.40mm_HandSolder, F.Cu at (130.1, 72.2)
- added R10: 4.7K, Resistor_SMD:R_0805_2012Metric_Pad1.15x1.40mm_HandSolder, F.Cu at (130.1, 66.3)
- added R11: 4.7K, Resistor_SMD:R_0805_2012Metric_Pad1.15x1.40mm_HandSolder, F.Cu at (116.8, 87.8)
- added R12: 4.7K, Resistor_SMD:R_0805_2012Metric_Pad1.15x1.40mm_HandSolder, F.Cu at (148.5, 122.7)
- added R13: 4.7K, Resistor_SMD:R_0805_2012Metric_Pad1.15x1.40mm_HandSolder, F.Cu at (110.1, 95.1)
- added R14: 220, Resistor_SMD:R_0805_2012Metric_Pad1.15x1.40mm_HandSolder, F.Cu at (105.3, 98.1)
- added R15: 10K, Resistor_SMD:R_0805_2012Metric_Pad1.15x1.40mm_HandSolder, F.Cu at (254.6, 146.2)
- added R16: 10K, Resistor_SMD:R_0805_2012Metric_Pad1.15x1.40mm_HandSolder, F.Cu at (161.9, 104.3)
- added R17: 10K, Resistor_SMD:R_0805_2012Metric_Pad1.15x1.40mm_HandSolder, F.Cu at (163.2, 113.2)
- added R18: 10K, Resistor_SMD:R_0805_2012Metric_Pad1.15x1.40mm_HandSolder, F.Cu at (163.2, 119.5)
- added R2: 100, Resistor_SMD:R_0805_2012Metric_Pad1.15x1.40mm_HandSolder, F.Cu at (120.6, 80.0)
- added R3: 100, Resistor_SMD:R_0805_2012Metric_Pad1.15x1.40mm_HandSolder, F.Cu at (130.1, 69.2)
- added R4: 4.7K, Resistor_SMD:R_0805_2012Metric_Pad1.15x1.40mm_HandSolder, F.Cu at (107.2, 92.2)
- added R5: 4.7K, Resistor_SMD:R_0805_2012Metric_Pad1.15x1.40mm_HandSolder, F.Cu at (124.2, 75.2)
- added R6: 240, Resistor_SMD:R_0805_2012Metric_Pad1.15x1.40mm_HandSolder, F.Cu at (227.9, 113.2)
- added R7: 240, Resistor_SMD:R_0805_2012Metric_Pad1.15x1.40mm_HandSolder, F.Cu at (227.9, 117.0)
- added R8: 240, Resistor_SMD:R_0805_2012Metric_Pad1.15x1.40mm_HandSolder, F.Cu at (227.9, 120.8)
- added R9: 240, Resistor_SMD:R_0805_2012Metric_Pad1.15x1.40mm_HandSolder, F.Cu at (227.9, 124.6)
- added SPND1: EBV-02-D, TerminalBlock:TerminalBlock_bornier-2_P5.08mm, F.Cu at (257.1, 153.8)
- added SW1: SW_Push, Button_Switch_SMD:SW_SPST_EVQPE1, F.Cu at (91.9, 83.8)
- added SX1: MOLEX_2031, Connector_Molex:Molex_KK-254_AE-6410-03A_1x03_P2.54mm_Vertical, F.Cu at (167.0, 104.3)
- added SY1: MOLEX_2031, Connector_Molex:Molex_KK-254_AE-6410-03A_1x03_P2.54mm_Vertical, F.Cu at (167.0, 111.9)
- added SZ1: MOLEX_2031, Connector_Molex:Molex_KK-254_AE-6410-03A_1x03_P2.54mm_Vertical, F.Cu at (167.0, 119.5)
- added U1: iCE40-HX4K-TQ144, Package_QFP:TQFP-144_20x20mm_P0.5mm, F.Cu at (193.7, 115.7)
- added U2: MCP1826S-3302E/DB, Package_TO_SOT_SMD:SOT-223, F.Cu at (149.2, 144.9)
- added U3: MCP1826S-1202E/DB, Package_TO_SOT_SMD:SOT-223, F.Cu at (164.4, 144.9)
- added U4: S25FL064LABMFI010, Package_SO:SOIJ-8_5.3x5.3mm_P1.27mm, F.Cu at (127.5, 46.0)
- added Y1: SIT8008BI-12-XXE-100, BeagleWire_elements_package:ASDMB-100.000MHZ-XY-T, F.Cu at (68.3, 82.5)
Connections:
- net /GPIO12(PWM0) renamed Net-(P1-Pad32)
- net /GPIO13(PWM1) renamed Net-(P1-Pad33)
- net /GPIO16 renamed Net-(P1-Pad36)
- net /GPIO18(GEN1)(PWM0) renamed Net-(P1-Pad12)
- net /GPIO23(GEN4) renamed Net-(P1-Pad16)
- net /GPIO24(GEN5) renamed Net-(P1-Pad18)
- net /GPIO25(GEN6) renamed Net-(P1-Pad22)
- net /GPIO26 renamed Net-(P1-Pad37)
- net /GPIO4(GCLK) renamed Net-(P1-Pad7)
- net /GPIO5 renamed Net-(P1-Pad29)
- net /GPIO6 renamed Net-(P1-Pad31)
- net /ID_SC renamed Net-(P1-Pad28)
- net /ID_SD renamed Net-(P1-Pad27)
- P1 pad 10: /GPIO15(RXD0) -> GPIO15
- P1 pad 11: /GPIO17(GEN0) -> ENABLE
- P1 pad 13: /GPIO27(GEN2) -> RP_CDONE
- P1 pad 15: /GPIO22(GEN3) -> RP_CRESET
- P1 pad 19: /GPIO10(SPI0_MOSI) -> SPI0_DI
- P1 pad 21: /GPIO9(SPI0_MISO) -> SPI0_DO
- P1 pad 23: /GPIO11(SPI0_SCK) -> SPI0_SCL
- P1 pad 24: /GPIO8(SPI0_CE_N) -> SPI0_CE
- P1 pad 26: /GPIO7(SPI1_CE_N) -> SPI1_CE
- P1 pad 3: /GPIO2(SDA1) -> POT_SDA
- P1 pad 35: /GPIO19(SPI1_MISO) -> SPI1_MISO
- P1 pad 38: /GPIO20(SPI1_MOSI) -> SPI1_MOSI
- P1 pad 40: /GPIO21(SPI1_SCK) -> SPI1_SCL
- P1 pad 5: /GPIO3(SCL1) -> POT_SCL
- P1 pad 8: /GPIO14(TXD0) -> GPIO14
Other:
- outline, holes or cut-outs redrawn
- board text removed: "CAMERA"
