File: base/extension/esp32.kicad_sch (KiCad schematic)
At the start: 6 parts, among them SW1 SW_Push_Open, SW2 SW_Push_Open, U2 ESP32-S3-WROOM-2

Commit message: changes for extension
Parts:
- removed D4: LED_ABGR, footprints:LED_Cree-PLCC4_2x2mm_CW, symbol Device:LED_ABGR
- removed SW2: SW_Push_Open, Button_Switch_SMD:SW_SPST_B3U-1000P, symbol Switch:SW_Push
- C9: Farnell 2094043 -> (none); Mouser 581-08055C105KAT2A -> (none); Producer 08055C105KAT2A -> (none)
- R4: Farnell 2826162 -> (none); Mouser 71-CRCW080510K0JNEAC -> (none); Producer CRCW080510K0JNEAC -> (none)
- SW1: footprint Button_Switch_SMD:SW_SPST_B3U-1000P -> footprints:SW_SPST_CK_KXT3; Farnell 1333652 -> 3023200; Mouser 653-B3U-1000P -> (none); Producer B3U-1000P -> (none)
- U2: Mouser ESP32-S3-WROOM-2-N32R8V -> (none); Producer ESP32-S3-WROOM-2-N32R8V -> (none)
Connections:
- net SPI_SS is gone; now on net POT_SCL: U2.18 (GPIO10/TOUCH10/ADC1_CH9/FSPICS0/FSPIIO4/SUBSPICS0)
- net CFG_DONE: now also U2.31 (GPIO38/FSPIWP/SUBSPIWP); no longer U2.25 (GPIO48/SPICLK_N/SUBSPICLK_N_DIFF)
- net POT_SCL: no longer U2.5 (GPIO5/TOUCH5/ADC1_CH4)
- net POT_SDA: now also U2.25 (GPIO48/SPICLK_N/SUBSPICLK_N_DIFF); no longer U2.4 (GPIO4/TOUCH4/ADC1_CH3)
- net SPI_SS_FPGA: now also U2.26 (GPIO45); no longer U2.17 (GPIO9/TOUCH9/ADC1_CH8/FSPIHD/SUBSPIHD)
- net SPI_SS_MOTOR: now also U2.35 (MTMS/GPIO42); no longer U2.22 (GPIO14/TOUCH14/ADC2_CH3/FSPIWP/FSPIDQS/SUBSPIWP)
- net STEP_ENABLE: now also U2.17 (GPIO9/TOUCH9/ADC1_CH8/FSPIHD/SUBSPIHD); no longer U2.31 (GPIO38/FSPIWP/SUBSPIWP)
- net Z_DIR: now reaches U2.23 (GPIO21)
- net FREE: now reaches U2.32 (MTCK/GPIO39/CLK_OUT3/SUBSPICS1)
- net SPI_SS_FLASH: now reaches U2.33 (MTDO/GPIO40/CLK_OUT2)
- net ESP32_BLUE: no longer names the net of U2.10 (GPIO17/U1TXD/ADC2_CH6)
- net ESP32_GREEN renamed Z_PO
- net ESP32_RED: no longer names the net of U2.12 (GPIO8/TOUCH8/ADC1_CH7/SUBSPICS1)
- net FPGA38: no longer names the net of U2.39 (GPIO1/TOUCH1/ADC1_CH0)
- net FPGA39: no longer names the net of U2.38 (GPIO2/TOUCH2/ADC1_CH1)
- net FPGA41: no longer names the net of U2.15 (GPIO3/TOUCH3/ADC1_CH2)
- net FPGA42: no longer names the net of U2.8 (GPIO15/U0RTS/ADC2_CH4/XTAL_32K_P)
- net FPGA43: no longer names the net of U2.9 (GPIO16/U0CTS/ADC2_CH5/XTAL_32K_N)
- net FPGA44 renamed SD_SS
- net FPGA46 renamed SD_MOSI
- net GPIO43 renamed Z_STEP
- net GPIO44: no longer names the net of U2.36 (U0RXD/GPIO44/CLK_OUT2)
- new net SD_CLK: U2.4 (GPIO4/TOUCH4/ADC1_CH3)
- new net SD_MISO: U2.5 (GPIO5/TOUCH5/ADC1_CH4)
- no-connect marks 7 -> 11
Other:
- note added: "ESP32"
- note removed: "GPIO 1 + 3 micropython REPL"
- note removed: "Microcontroller"
- note removed: "Microcontroller light"
- company: Hexastorm -> (none)
- title: Firestarter  -> (none)
- moved on the sheet: R4, SW1, U2
