File: lasermodule/felixmount/felixmount.kicad_sch (KiCad schematic)
At the start: 4 parts

Commit message: sent to pcbway
Parts:
- added H5, H6, H7, H8: MountingHole, MountingHole:MountingHole_6.4mm_M6, symbol Mechanical:MountingHole
Other:
- note added: "connections laser base"
- note added: "connections optical plate 25 mm pitch, m6"
