File: base/esp32.kicad_sch (KiCad schematic)
At the start: 7 parts, among them SW1 SW_Push_Open, SW2 SW_Push_Open, U2 ESP32-S3-WROOM-2

Commit message: added comment chip, changed i2c resistor to 1.5K
Parts:
- R8, R9: value 5.1K -> 1.5K; manf# CRCW08055K10FKEA -> CR0805-JW-152ELF; mouser# -71-CRCW0805-5.1K-E3 -> 652-CR0805JW-152ELF
Changed lines of the file:
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@@
 			)
 		)
-		(property "Value" "5.1K"
+		(property "Value" "1.5K"
 			(at 232.41 67.564 0)
 			(show_name no)
@@
 			)
 		)
-		(property "manf#" "CRCW08055K10FKEA"
+		(property "manf#" "CR0805-JW-152ELF"
 			(at 238.76 66.04 0)
 			(hide yes)
@@
 			)
 		)
-		(property "mouser#" "-71-CRCW0805-5.1K-E3"
+		(property "mouser#" "652-CR0805JW-152ELF"
 			(at 238.76 66.04 0)
 			(hide yes)
@@
 			)
 		)
-		(property "Value" "5.1K"
+		(property "Value" "1.5K"
 			(at 241.3 67.564 0)
 			(show_name no)
@@
 			)
 		)
-		(property "manf#" "CRCW08055K10FKEA"
+		(property "manf#" "CR0805-JW-152ELF"
 			(at 247.65 66.04 0)
 			(hide yes)
@@
 			)
 		)
-		(property "mouser#" "-71-CRCW0805-5.1K-E3"
+		(property "mouser#" "652-CR0805JW-152ELF"
 			(at 247.65 66.04 0)
 			(hide yes)
