File: base/compute.kicad_pcb (KiCad board)
At the start: 4 copper layers, 88.4 x 63.6 mm, 125 parts, among them IC1 TMC2209-LA-T, IC2 TMC2209-LA-T, IC3 TMC2209-LA-T, IC4 DMP6023LSS-13, J1 USB_C_Receptacle_USB2.0_16P, J13 fan, J2 FPC-24P-0.5mm, J3 2-84952-0, J4 DC_Jack_5.5x2.5, J9 spindle, Q1 Q_NMOS_GDS_spindle, Q2 Q_NMOS_GSD_fan, SW1 SW_Push_Open, SW2 SW_Push_Open, U1 MCP1700T-1202ETT, U2 ESP32-S3-WROOM-2, U3 LM1117MPX-5.0/NOPB, U4 MCP1700-1502, U5 ICE40UP5K-SG48ITR-FPGA_Lattice, U6 MCP1700T-2802E, U7 USBLC6-2SC6, U8 AP63203WU-7

Commit message: improved ability for optical inpspection usb connector and motors
Parts:
- moved R26 19.2 mm to (173.0, 183.5)
- moved D1 17.3 mm to (172.9, 180.7)
- moved C26 10.3 mm to (177.6, 166.9), turned to 0 degrees
- moved IC4 7.18 mm to (175.9, 175.9)
- moved C27 4.67 mm to (227.5, 150.8)
- moved D4 3.54 mm to (188.0, 163.4), turned to 180 degrees
- moved IC3 3.15 mm to (230.5, 176.1)
- moved IC2 3.00 mm to (230.5, 162.3)
- moved IC1 2.74 mm to (230.9, 146.1)
- moved G1 1.35 mm to (221.8, 142.4)
- moved F1 1.21 mm to (173.4, 187.7)
- moved C22 1.20 mm to (233.7, 150.7)
- moved FB1 1.18 mm to (173.1, 185.5)
- moved C34 0.54 mm to (231.6, 157.6)
- turned C25 to 0 degrees
Routing:
- net +24V: track 449.3 -> 462.2 mm
- net +3.3V: track 270.5 -> 283.1 mm, vias 8 -> 5
- net GND: track 257.8 -> 245.3 mm, vias 36 -> 38
- net Net-(D4-A1): track 29.6 -> 21.1 mm
- net Y_DIR: track 25.6 -> 17.9 mm
- net DIAG_Y: track 15.9 -> 10.6 mm, vias 0 -> 2
- net Z_DIR: track 35.1 -> 30.1 mm
- net X_DIR: track 28.1 -> 23.4 mm
- net Y_STEP: track 20.1 -> 15.6 mm
- net Z_STEP: track 32.3 -> 28.0 mm
- net UARX: track 92.8 -> 88.6 mm
- net Z_A1: track 15.1 -> 18.3 mm
- net Z_B1: track 15.9 -> 19.0 mm
- net DIAG_Z: track 24.6 -> 21.4 mm
- net Z_A2: track 18.8 -> 22.0 mm
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
Commit message: small fix compute pcb
Parts:
- J2: value FPC-24P-0.5mm -> FH12A-24S-0.5SH
- J4: footprint footprints:BarrelJack_CUI_PJ-036AH-SMT_Horizontal -> Connector_BarrelJack:BarrelJack_CUI_PJ-079BH_Horizontal
- R8, R9: value 5.1K -> 1.5K
- moved J4 4.00 mm to (200.5, 183.8)
Routing:
- net Net-(F2-Pad2): track 8.49 -> 15.8 mm
- net GND: vias 38 -> 37
