File: base/compute.kicad_sch (KiCad schematic)
At the start: 52 parts, among them IC4 DMP6023LSS-13, J1 USB_C_Receptacle_USB2.0_16P, J3 2-84952-0, J4 DC_Jack_5.5x2.5, U1 MCP1700T-1202ETT, U3 LM1117MPX-5.0/NOPB, U4 MCP1700-1502, U6 MCP1700T-2802E, U7 USBLC6-2SC6, U8 AP63203WU-7

Commit message: added comment chip, changed i2c resistor to 1.5K
Parts:
- C56: farnell# 718567 -> 3606028; manf# CC0805JRNPO9BN102 -> C0805JRNPO9BN101; mouser# 603-CC805JRNPO9BN102 -> 603-CC805JRNPO9BN101
Changed lines of the file:
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@@
 			)
 		)
-		(property "manf#" "CC0805JRNPO9BN102"
+		(property "manf#" "C0805JRNPO9BN101"
 			(at 102.87 139.7 0)
 			(hide yes)
@@
 			)
 		)
-		(property "mouser#" "603-CC805JRNPO9BN102"
+		(property "mouser#" "603-CC805JRNPO9BN101"
 			(at 102.87 139.7 0)
 			(hide yes)
@@
 			)
 		)
-		(property "farnell#" "718567"
+		(property "farnell#" "3606028"
 			(at 102.87 139.7 0)
 			(hide yes)

Commit message: small fix compute pcb
Parts:
- J4: footprint footprints:BarrelJack_CUI_PJ-036AH-SMT_Horizontal -> Connector_BarrelJack:BarrelJack_CUI_PJ-079BH_Horizontal; farnell# 4814432 -> 4814468; manf# PJ-036BH-SMT-TR -> PJ-079BH; mouser# 490-PJ-036BH-SMT-TR -> 490-PJ-079BH
Changed lines of the file:
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@@
 			)
 		)
-		(property "Footprint" "footprints:BarrelJack_CUI_PJ-036AH-SMT_Horizontal"
+		(property "Footprint" "Connector_BarrelJack:BarrelJack_CUI_PJ-079BH_Horizontal"
 			(at 72.39 28.956 0)
 			(hide yes)
@@
 			)
 		)
-		(property "manf#" "PJ-036BH-SMT-TR"
+		(property "manf#" "PJ-079BH "
 			(at 71.12 27.94 0)
 			(hide yes)
@@
 			)
 		)
-		(property "mouser#" "490-PJ-036BH-SMT-TR"
+		(property "mouser#" "490-PJ-079BH"
 			(at 71.12 27.94 0)
 			(hide yes)
@@
 			)
 		)
-		(property "farnell#" "4814432"
+		(property "farnell#" "4814468"
 			(at 71.12 27.94 0)
 			(hide yes)
