File: lasermodule/connectorplate/plate.kicad_sch (KiCad schematic)
At the start: 2 parts, among them J1 292173-5, J2 Conn_01x05

Commit message: Outside of the format migration, there are only minor component/footprint updates:
base.kicad_sch
J2: Marked as Do Not Populate ((dnp yes)).
J2 footprint: Switched from custom library to standard KiCad library: sockets_scanhead:motor_13pin → Connector_PinSocket_2.00mm:PinSocket_1x13_P2.00mm_Vertical

plate.kicad_sch
Connector footprint: Switched to standard library: mirrormotor:PinHeader_1x05_P2.00mm_Vertical → Connector_PinHeader_2.00mm:PinHeader_1x05_P2.00mm_Vertical
Part order numbers added: Added #manf: M22-2510505, #mouser: 855-M22-2510505, and #farnell: 3226026.
No-connect: Added a (no_connect) symbol on pin coordinate (109.22, 81.28).

mirrormotor.kicad_sch
0 circuit changes: Exactly 4 lines changed outside lib_symbols (the version header). All ~1,486 other lines are symbol cache syntax additions.
Parts:
- J2: footprint mirrormotor:PinHeader_1x05_P2.00mm_Vertical -> Connector_PinHeader_2.00mm:PinHeader_1x05_P2.00mm_Vertical; #farnell (none) -> 3226026; #manf (none) -> M22-2510505; #mouser (none) -> 855-M22-2510505
Changed lines of the file:
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@@
 (kicad_sch
-	(version 20231120)
+	(version 20260306)
 	(generator "eeschema")
-	(generator_version "8.0")
+	(generator_version "10.0")
 	(paper "A4")
+	(text "GND\n"
+		(exclude_from_sim no)
+		(at 78.74 91.694 0)
+		(effects
+			(font
+				(size 1.27 1.27)
+			)
+		)
+	)
+	(text "12V"
+		(exclude_from_sim no)
+		(at 78.994 86.36 0)
+		(effects
+			(font
+				(size 1.27 1.27)
+			)
+		)
+	)
+	(text "Ricoh AF-1027/270 using NBC3111 chip"
+		(exclude_from_sim no)
+		(at 66.04 81.026 0)
+		(effects
+			(font
+				(size 1.27 1.27)
+			)
+		)
+	)
+	(text "PWM"
+		(exclude_from_sim no)
+		(at 78.74 96.52 0)
+		(effects
+			(font
+				(size 1.27 1.27)
+			)
+		)
+	)
+	(text "GND\n"
+		(exclude_from_sim no)
+		(at 78.74 89.154 0)
+		(effects
+			(font
+				(size 1.27 1.27)
+			)
+		)
+	)
+	(text "NC"
+		(exclude_from_sim no)
+		(at 78.74 93.98 0)
+		(effects
+			(font
+				(size 1.27 1.27)
+			)
+		)
+	)
 	(no_connect
 		(at 109.22 81.28)
@@
 			(width 0)
 			(type default)
-		)
-	)
-	(text "GND\n"
-		(exclude_from_sim no)
-		(at 78.74 91.694 0)
-		(effects
-			(font
-				(size 1.27 1.27)
-			)
-		)
-	)
-	(text "12V"
-		(exclude_from_sim no)
-		(at 78.994 86.36 0)
-		(effects
-			(font
-				(size 1.27 1.27)
-			)
-		)
-	)
-	(text "Ricoh AF-1027/270 using NBC3111 chip"
-		(exclude_from_sim no)
-		(at 66.04 81.026 0)
-		(effects
-			(font
-				(size 1.27 1.27)
-			)
-		)
-	)
-	(text "PWM"
-		(exclude_from_sim no)
-		(at 78.74 96.52 0)
-		(effects
-			(font
-				(size 1.27 1.27)
-			)
-		)
-	)
-	(text "GND\n"
-		(exclude_from_sim no)
-		(at 78.74 89.154 0)
-		(effects
-			(font
-				(size 1.27 1.27)
-			)
-		)
-	)
-	(text "NC"
-		(exclude_from_sim no)
-		(at 78.74 93.98 0)
-		(effects
-			(font
-				(size 1.27 1.27)
-			)
 		)
 	)
@@
 		(mirror x)
 		(unit 1)
+		(body_style 1)
 		(exclude_from_sim no)
 		(in_bom yes)
 		(on_board yes)
+		(in_pos_files yes)
 		(dnp no)
 		(fields_autoplaced yes)
 		(property "Reference" "J1"
 			(at 111.76 89.8143 0)
+			(show_name no)
+			(do_not_autoplace no)
 			(effects
 				(font
@@
 		(property "Value" "292173-5"
 			(at 111.76 92.3543 0)
+			(show_name no)
+			(do_not_autoplace no)
 			(effects
 				(font
@@
 		(property "Footprint" "mirrormotor:2921735"
 			(at 109.22 91.44 0)
-			(effects
-				(font
-					(size 1.27 1.27)
-				)
-				(hide yes)
-			)
-		)
-		(property "Datasheet" "~"
+			(hide yes)
+			(show_name no)
+			(do_not_autoplace no)
+			(effects
+				(font
+					(size 1.27 1.27)
+				)
+			)
+		)
+		(property "Datasheet" ""
 			(at 109.22 91.44 0)
-			(effects
-				(font
-					(size 1.27 1.27)
-				)
-				(hide yes)
+			(hide yes)
+			(show_name no)
+			(do_not_autoplace no)
+			(effects
+				(font
+					(size 1.27 1.27)
+				)
 			)
 		)
 		(property "Description" "Generic connectable mounting pin connector, single row, 01x05, script generated (kicad-library-utils/schlib/autogen/connector/)"
 			(at 109.22 91.44 0)
-			(effects
-				(font
-					(size 1.27 1.27)
-				)
-				(hide yes)
+			(hide yes)
+			(show_name no)
+			(do_not_autoplace no)
+			(effects
+				(font
+					(size 1.27 1.27)
+				)
 			)
 		)
@@
 		(at 93.98 91.44 180)
 		(unit 1)
+		(body_style 1)
 		(exclude_from_sim no)
 		(in_bom yes)
 		(on_board yes)
+		(in_pos_files yes)
 		(dnp no)
 		(fields_autoplaced yes)
 		(property "Reference" "J2"
 			(at 87.63 91.44 90)
+			(show_name no)
+			(do_not_autoplace no)
 			(effects
 				(font
@@
 		(property "Value" "Conn_01x05"
 			(at 90.17 91.44 90)
-			(effects
-				(font
-					(size 1.27 1.27)
-				)
-			)
-		)
-		(property "Footprint" "mirrormotor:PinHeader_1x05_P2.00mm_Vertical"
+			(show_name no)
+			(do_not_autoplace no)
+			(effects
+				(font
+					(size 1.27 1.27)
+				)
+			)
+		)
+		(property "Footprint" "Connector_PinHeader_2.00mm:PinHeader_1x05_P2.00mm_Vertical"
 			(at 93.98 91.44 0)
-			(effects
-				(font
-					(size 1.27 1.27)
-				)
-				(hide yes)
-			)
-		)
-		(property "Datasheet" "~"
+			(hide yes)
+			(show_name no)
+			(do_not_autoplace no)
+			(effects
+				(font
+					(size 1.27 1.27)
+				)
+			)
+		)
+		(property "Datasheet" ""
 			(at 93.98 91.44 0)
-			(effects
-				(font
-					(size 1.27 1.27)
-				)
-				(hide yes)
+			(hide yes)
+			(show_name no)
+			(do_not_autoplace no)
+			(effects
+				(font
+					(size 1.27 1.27)
+				)
 			)
 		)
 		(property "Description" "Generic connector, single row, 01x05, script generated (kicad-library-utils/schlib/autogen/connector/)"
 			(at 93.98 91.44 0)
-			(effects
-				(font
-					(size 1.27 1.27)
-				)
-				(hide yes)
+			(hide yes)
+			(show_name no)
+			(do_not_autoplace no)
+			(effects
+				(font
+					(size 1.27 1.27)
+				)
+			)
+		)
+		(property "#manf" "M22-2510505"
+			(at 93.98 91.44 90)
+			(hide yes)
+			(show_name no)
+			(do_not_autoplace no)
+			(effects
+				(font
+					(size 1.27 1.27)
+				)
+			)
+		)
+		(property "#mouser" "855-M22-2510505"
+			(at 93.98 91.44 90)
+			(hide yes)
+			(show_name no)
+			(do_not_autoplace no)
+			(effects
+				(font
+					(size 1.27 1.27)
+				)
+			)
+		)
+		(property "#farnell" "3226026"
+			(at 93.98 91.44 90)
+			(hide yes)
+			(show_name no)
+			(do_not_autoplace no)
+			(effects
+				(font
+					(size 1.27 1.27)
+				)
 			)
 		)
@@
 		)
 		(instances
-			(project ""
+			(project "plate"
 				(path "/593d3fe2-52a4-4dc3-98a9-0f815bbe0b09"
 					(reference "J2")
@@
 		)
 	)
+	(embedded_fonts no)
 )
