File: lasermodule/backplate/backplate.kicad_pcb (KiCad board)
At the start: 2 copper layers, 24.2 x 54.1 mm, 5 parts, among them J1 Conn_01x01, J2 Conn_01x01, J3 Conn_01x01, J4 Conn_01x01, J5 Conn_01x02

Commit message: updated pcbs
Parts:
- moved J4 0.97 mm to (142.8, 120.2)
- moved J1 0.97 mm to (142.9, 87.6)
- moved J3 0.96 mm to (165.4, 120.2)
- moved J2 0.95 mm to (165.4, 87.7)
- moved J5 0.71 mm to (155.9, 103.9)
Routing:
- net +12V: track 29.1 -> 32.4 mm
Other:
- board size 24.2 x 54.1 mm -> 25.7 x 54.1 mm
