File: lasermodule/base/laserhead.kicad_sch (KiCad schematic)
At the start: 25 parts, among them J1 fan laser, J13 Conn_01x01, J14 Conn_01x01, U1 DIGIPOT_50K, U2 U_IC-HKB, U4 MIC920, U5 MIC920

Commit message: added comment chip, changed i2c resistor to 1.5K
Other:
- note added: "TTL is op 3.3V je moet chip met 3.3V voeden"
Changed lines of the file:
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@@
+		)
+	)
+	(text "TTL is op 3.3V je moet chip met 3.3V voeden"
+		(exclude_from_sim no)
+		(at 108.458 54.356 0)
+		(effects
+			(font
+				(size 1.27 1.27)
+			)
 		)
 	)

Commit message: updated pcbs
Parts:
- U4, U5: footprint Package_TO_SOT_SMD:SOT-353_SC-70-5_Handsoldering -> Package_TO_SOT_SMD:SOT-353_SC-70-5
Changed lines of the file:
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@@
 			)
 		)
-		(property "Footprint" "Package_TO_SOT_SMD:SOT-353_SC-70-5_Handsoldering"
+		(property "Footprint" "Package_TO_SOT_SMD:SOT-353_SC-70-5"
 			(at 203.2 69.85 0)
 			(hide yes)
@@
 			)
 		)
-		(property "Footprint" "Package_TO_SOT_SMD:SOT-353_SC-70-5_Handsoldering"
+		(property "Footprint" "Package_TO_SOT_SMD:SOT-353_SC-70-5"
 			(at 232.41 69.85 0)
 			(hide yes)
