File: lasermodule/base/base.kicad_sch (KiCad schematic)
At the start: 18 parts, among them J10 Conn_01x01, J11 Conn_01x01, J12 Conn_01x01, J19 2-84952-0, J2 Conn_01x13, J6 mirrormotor, J7 Conn_01x01, J8 Conn_01x01, J9 Conn_01x01

Commit message: Outside of the format migration, there are only minor component/footprint updates:
base.kicad_sch
J2: Marked as Do Not Populate ((dnp yes)).
J2 footprint: Switched from custom library to standard KiCad library: sockets_scanhead:motor_13pin → Connector_PinSocket_2.00mm:PinSocket_1x13_P2.00mm_Vertical

plate.kicad_sch
Connector footprint: Switched to standard library: mirrormotor:PinHeader_1x05_P2.00mm_Vertical → Connector_PinHeader_2.00mm:PinHeader_1x05_P2.00mm_Vertical
Part order numbers added: Added #manf: M22-2510505, #mouser: 855-M22-2510505, and #farnell: 3226026.
No-connect: Added a (no_connect) symbol on pin coordinate (109.22, 81.28).

mirrormotor.kicad_sch
0 circuit changes: Exactly 4 lines changed outside lib_symbols (the version header). All ~1,486 other lines are symbol cache syntax additions.
Parts:
- J2: footprint sockets_scanhead:motor_13pin -> Connector_PinSocket_2.00mm:PinSocket_1x13_P2.00mm_Vertical; now not fitted
Changed lines of the file:
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@@
 		(on_board yes)
 		(in_pos_files yes)
-		(dnp no)
+		(dnp yes)
 		(property "Reference" "J2"
 			(at 187.96 60.9599 0)
@@
 			)
 		)
-		(property "Footprint" "sockets_scanhead:motor_13pin"
+		(property "Footprint" "Connector_PinSocket_2.00mm:PinSocket_1x13_P2.00mm_Vertical"
 			(at 185.42 62.23 0)
 			(hide yes)

Commit message: maxwell lock updated, magnets cutouts improved
Parts:
- added MAG1, MAG2, MAG3: Magnet_D8x2mm, sockets_scanhead:TestPoint_Pad_D8.0mm, symbol Connector:TestPoint
Connections:
- no-connect marks 6 -> 9
Changed lines of the file:
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@@
 		(color 0 0 0 0)
 	)
+		(no_connect
+		(at 134.62 104.14)
+	)
+	(no_connect
+		(at 152.4 104.14)
+	)
 	(no_connect
+		(at 170.18 104.14)
+	)
+(no_connect
 		(at 95.25 59.69)
 	)
@@
 	)
 	(symbol
+		(lib_id "Connector:TestPoint")
+		(at 170.18 104.14 0)
+		(unit 1)
+		(body_style 1)
+		(exclude_from_sim no)
+		(in_bom yes)
+		(on_board yes)
+		(in_pos_files yes)
+		(dnp no)
+		(property "Reference" "MAG3"
+			(at 170.18 96.52 0)
+			(show_name no)
+			(do_not_autoplace no)
+			(effects
+				(font
+					(size 1.27 1.27)
+				)
+			)
+		)
+		(property "Value" "Magnet_D8x2mm"
+			(at 170.18 98.425 0)
+			(show_name no)
+			(do_not_autoplace no)
+			(effects
+				(font
+					(size 1.27 1.27)
+				)
+			)
+		)
+		(property "Footprint" "sockets_scanhead:TestPoint_Pad_D8.0mm"
+			(at 175.26 104.14 0)
+			(hide yes)
+			(show_name no)
+			(do_not_autoplace no)
+			(effects
+				(font
+					(size 1.27 1.27)
+				)
+			)
+		)
+		(property "Datasheet" ""
+			(at 175.26 104.14 0)
+			(hide yes)
+			(show_name no)
+			(do_not_autoplace no)
+			(effects
+				(font
+					(size 1.27 1.27)
+				)
+			)
+		)
+		(property "Description" "Neodymium Magnet Ø8x2mm"
+			(at 170.18 104.14 0)
+			(hide yes)
+			(show_name no)
+			(do_not_autoplace no)
+			(effects
+				(font
+					(size 1.27 1.27)
+				)
+			)
+		)
+		(pin "1"
+		)
+		(instances
+			(project "base"
+				(path "/e63e39d7-6ac0-4ffd-8aa3-1841a4541b55"
+					(reference "MAG3")
+					(unit 1)
+				)
+			)
+		)
+	)
+	(symbol
 		(lib_id "power:+5V")
 		(at 41.91 76.2 90)
@@
 	)
 	(symbol
+		(lib_id "Connector:TestPoint")
+		(at 152.4 104.14 0)
+		(unit 1)
+		(body_style 1)
+		(exclude_from_sim no)
+		(in_bom yes)
+		(on_board yes)
+		(in_pos_files yes)
+		(dnp no)
+		(property "Reference" "MAG2"
+			(at 152.4 96.52 0)
+			(show_name no)
+			(do_not_autoplace no)
+			(effects
+				(font
+					(size 1.27 1.27)
+				)
+			)
+		)
+		(property "Value" "Magnet_D8x2mm"
+			(at 152.4 98.425 0)
+			(show_name no)
+			(do_not_autoplace no)
+			(effects
+				(font
+					(size 1.27 1.27)
+				)
+			)
+		)
+		(property "Footprint" "sockets_scanhead:TestPoint_Pad_D8.0mm"
+			(at 157.48 104.14 0)
+			(hide yes)
+			(show_name no)
+			(do_not_autoplace no)
+			(effects
+				(font
+					(size 1.27 1.27)
+				)
+			)
+		)
+		(property "Datasheet" ""
+			(at 157.48 104.14 0)
+			(hide yes)
+			(show_name no)
+			(do_not_autoplace no)
+			(effects
+				(font
+					(size 1.27 1.27)
+				)
+			)
+		)
+		(property "Description" "Neodymium Magnet Ø8x2mm"
+			(at 152.4 104.14 0)
+			(hide yes)
+			(show_name no)
+			(do_not_autoplace no)
+			(effects
+				(font
+					(size 1.27 1.27)
+				)
+			)
+		)
+		(pin "1"
+		)
+		(instances
+			(project "base"
+				(path "/e63e39d7-6ac0-4ffd-8aa3-1841a4541b55"
+					(reference "MAG2")
+					(unit 1)
+				)
+			)
+		)
+	)
+	(symbol
 		(lib_id "Mechanical:MountingHole")
 		(at 96.52 106.68 0)
@@
 					(unit 1)
 				)
+			)
+		)
+	)
+	(symbol
+		(lib_id "Connector:TestPoint")
+		(at 134.62 104.14 0)
+		(unit 1)
+		(body_style 1)
+		(exclude_from_sim no)
+		(in_bom yes)
+		(on_board yes)
+		(in_pos_files yes)
+		(dnp no)
+		(property "Reference" "MAG1"
+			(at 134.62 96.52 0)
+			(show_name no)
+			(do_not_autoplace no)
+			(effects
+				(font
+					(size 1.27 1.27)
+				)
+			)
+		)
+		(property "Value" "Magnet_D8x2mm"
+			(at 134.62 98.425 0)
+			(show_name no)
+			(do_not_autoplace no)
+			(effects
+				(font
+					(size 1.27 1.27)
+				)
+			)
+		)
+		(property "Footprint" "sockets_scanhead:TestPoint_Pad_D8.0mm"
+			(at 139.7 104.14 0)
+			(hide yes)
+			(show_name no)
+			(do_not_autoplace no)
+			(effects
+				(font
+					(size 1.27 1.27)
+				)
+			)
+		)
+		(property "Datasheet" ""
+			(at 139.7 104.14 0)
+			(hide yes)
+			(show_name no)
+			(do_not_autoplace no)
+			(effects
+				(font
+					(size 1.27 1.27)
+				)
+			)
+		)
+		(property "Description" "Neodymium Magnet Ø8x2mm"
+			(at 134.62 104.14 0)
+			(hide yes)
+			(show_name no)
+			(do_not_autoplace no)
+			(effects
+				(font
+					(size 1.27 1.27)
+				)
+			)
+		)
+		(pin "1"
+		)
+		(instances
+			(project "base"
+				(path "/e63e39d7-6ac0-4ffd-8aa3-1841a4541b55"
+					(reference "MAG1")
+					(unit 1)
+				)
