File: lasermodule/laserdiode/laserdiode.kicad_pcb (KiCad board)
At the start: 2 copper layers, 33.3 x 15.5 mm, 15 parts, among them J1 Conn_01x04, J2 Conn_01x01, J3 Conn_01x01, J4 Conn_01x01, J5 Conn_01x01, J6 Conn_01x01, J7 Conn_01x01

Commit message: updated pcbs
Parts:
- removed J6, J7: Conn_01x01, laserdiode:23765912
Routing:
- net unconnected-(J6-Pin_1-Pad1): track 5.68 -> 0.00 mm
- net unconnected-(J7-Pin_1-Pad1): track 5.54 -> 0.00 mm
Other:
- board size 33.3 x 15.5 mm -> 21 x 15.5 mm
- board text removed: "magnet strip"
