File: lasermodule/laserdiode/laserdiode.kicad_sch (KiCad schematic)
At the start: 15 parts, among them J1 Conn_01x04, J2 Conn_01x01, J3 Conn_01x01, J4 Conn_01x01, J5 Conn_01x01, J6 Conn_01x01, J7 Conn_01x01

Commit message: updated pcbs
Parts:
- removed J6, J7: Conn_01x01, laserdiode:23765912, symbol Connector_Generic:Conn_01x01
Connections:
- no-connect marks 2 -> 0
