File: lasermodule/sideplatediode/sideplatediode.kicad_pcb (KiCad board)
At the start: 2 copper layers, 99.8 x 24.2 mm, 7 parts, among them J2 Conn_01x01, J3 Conn_01x01, J4 Conn_01x01, J5 Conn_01x01

Commit message: updated pcbs
Parts:
- moved D1 1.22 mm to (108.5, 99.0)
- moved J3 0.97 mm to (159.6, 89.7)
- moved J2 0.95 mm to (142.3, 89.8)
- moved J4 0.93 mm to (190.3, 112.3)
- moved J5 0.91 mm to (111.7, 112.3)
Routing:
- net DiodeK: track 8.91 -> 11.6 mm
Other:
- board size 99.8 x 24.2 mm -> 99.8 x 25.7 mm
- board text added: "photodiode"
- board text removed: "pos1"
- board text removed: "pos2"
