File: lasermodule/sideplatediode/sideplatediode.kicad_sch (KiCad schematic)
At the start: 7 parts, among them J2 Conn_01x01, J3 Conn_01x01, J4 Conn_01x01, J5 Conn_01x01

Commit message: updated pcbs
Parts:
- D1: footprint DIO_BPW_34_S-Z -> start-of-scanline-detector:DIO_BPW_34_S-Z
